File: NodeMCU_Emon.brd (EAGLE design)
At the start: 73 x 44.7 mm, 19 parts, among them IC1 7805T, J3 10p-2.54, J4 4P-2.0, J5 DC-005, X1 STEREOJACK

Commit message: Added extra resistor to protect ADC
Parts:
- added R5: 10K, resistor:0204/7
- C2: value 10uF -> 100uF
- R2: value 22K -> 100K
- moved R2 0.76 mm to (56.8, 22.1)
- renumbered IC1 to IC1-D24V5F5
Connections:
- net V_AC renamed V_AC+
- removed net N$2: B1.AC1, J5.+, R3.2
- new net A2: J3.9, R5.1
- new net V_AC-: B1.AC1, J5.+, R3.2, R5.2
- net GND: no longer J3.9
- net N$3: now also J5.-1; no longer J5.-2
Routing:
- net V_AC-: track 0.00 -> 23.5 mm
- net N$2: track 16.9 -> 0.00 mm
- net A2: track 0.00 -> 16.0 mm
- net N$3: track 17.9 -> 21.7 mm
Changed lines of the file:
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@@
 <attribute name="NAME" x="50.165" y="41.148" size="1.27" layer="33" ratio="10" rot="R180"/>
 </element>
-<element name="J5" library="Seeed-OPL-Connector" package="DCJ3P-14.2X11.0X9.0MM" value="DC-005" x="64.135" y="10.922" rot="R180">
+<element name="J5" library="Seeed-OPL-Connector" package="DCJ3P-14.2X11.0X9.0MM" value="DC-005" x="64.135" y="10.922" smashed="yes" rot="R180">
 <attribute name="MPN" value="DC-005" x="64.135" y="10.922" size="1.778" layer="27" rot="R180" display="off"/>
-</element>
-<element name="R2" library="resistor" package="0204/7" value="22K" x="56.769" y="22.86"/>
+<attribute name="NAME" x="69.723" y="7.239" size="0.889" layer="25" ratio="11" rot="R180"/>
+<attribute name="VALUE" x="73.66" y="11.557" size="0.889" layer="27" ratio="11" rot="R180"/>
+<attribute name="NAME" x="64.135" y="11.557" size="0.254" layer="33" ratio="10" rot="R270"/>
+</element>
+<element name="R2" library="resistor" package="0204/7" value="100K" x="56.769" y="22.098" smashed="yes">
+<attribute name="NAME" x="61.722" y="21.4884" size="0.9906" layer="25" ratio="10"/>
+<attribute name="VALUE" x="55.1434" y="21.6154" size="0.9906" layer="27" ratio="10"/>
+</element>
 <element name="R3" library="resistor" package="0204/7" value="10K" x="56.769" y="19.431" rot="R180"/>
 <element name="R4" library="resistor" package="0204/7" value="330R" x="56.007" y="32.258" rot="R90"/>
 <element name="X1" library="adafruit" package="STX3100" value="STEREOJACK" x="71.247" y="32.258" smashed="yes" rot="R180">
-<attribute name="NAME" x="61.134" y="25.5" size="1.27" layer="25" ratio="10" rot="R180"/>
+<attribute name="NAME" x="67.103" y="25.373" size="1.27" layer="25" ratio="10" rot="R180"/>
 <attribute name="VALUE" x="69.897" y="39.978" size="1.27" layer="27" ratio="10" rot="R180"/>
 </element>
 <element name="C1" library="adafruit" package="TT2D4" value="10uF" x="42.926" y="7.747" rot="R270"/>
-<element name="C2" library="adafruit" package="TT2D4" value="10uF" x="42.926" y="13.97" rot="R90"/>
-<element name="IC1" library="adafruit" package="TO220H" value="7805T" x="45.085" y="30.099" smashed="yes">
-<attribute name="NAME" x="52.324" y="25.019" size="1.778" layer="25" ratio="10" rot="R90"/>
+<element name="C2" library="adafruit" package="TT2D4" value="100uF" x="42.926" y="13.97" rot="R90"/>
+<element name="IC1-D24V5F5" library="adafruit" package="TO220H" value="7805T" x="45.085" y="30.099" smashed="yes">
+<attribute name="NAME" x="52.197" y="21.209" size="1.778" layer="25" ratio="10" rot="R90"/>
 <attribute name="VALUE" x="52.451" y="19.05" size="1.778" layer="27" ratio="10" rot="R90"/>
 </element>
 <element name="B1" library="rectifier" package="B-DIL" value="" x="51.816" y="12.065" rot="R270"/>
 <element name="J4" library="Seeed-OPL-Connector" package="HW4-2.0" value="4P-2.0" x="58.166" y="3.556"/>
+<element name="R5" library="resistor" package="0204/7" value="10K" x="56.769" y="24.892" smashed="yes" rot="R180">
+<attribute name="NAME" x="63.5" y="25.3746" size="0.9906" layer="25" ratio="10" rot="R180"/>
+<attribute name="VALUE" x="58.3946" y="25.3746" size="0.9906" layer="27" ratio="10" rot="R180"/>
+</element>
 </elements>
 <signals>
@@
 <via x="11.43" y="36.83" extent="1-16" drill="0.3048" diameter="0.635"/>
 <contactref element="C2" pad="-"/>
-<contactref element="IC1" pad="2"/>
+<contactref element="IC1-D24V5F5" pad="2"/>
 <contactref element="B1" pad="-"/>
 <contactref element="C1" pad="-"/>
 <contactref element="J3" pad="2"/>
-<contactref element="J3" pad="9"/>
 <contactref element="J4" pad="4"/>
 </signal>
@@
 <contactref element="J13" pad="15"/>
 <wire x1="6.477" y1="4.699" x2="9.017" y2="4.699" width="0.8128" layer="1"/>
-<contactref element="IC1" pad="3"/>
+<contactref element="IC1-D24V5F5" pad="3"/>
 <contactref element="C2" pad="+"/>
 <wire x1="42.9768" y1="13.4112" x2="42.9768" y2="12.7254" width="0.8128" layer="16"/>
@@
 <contactref element="J3" pad="4"/>
 <contactref element="J4" pad="2"/>
-<wire x1="57.15" y1="24.4602" x2="57.15" y2="3.5814" width="0.1524" layer="16"/>
-<wire x1="48.8442" y1="32.766" x2="57.15" y2="24.4602" width="0.1524" layer="16"/>
+<wire x1="57.15" y1="10.4394" x2="57.15" y2="3.5814" width="0.1524" layer="16"/>
+<wire x1="48.8442" y1="18.7452" x2="57.15" y2="10.4394" width="0.1524" layer="16"/>
 <wire x1="48.8442" y1="40.4622" x2="48.8442" y2="37.5666" width="0.1524" layer="16"/>
-<wire x1="48.8442" y1="37.5666" x2="48.8442" y2="32.766" width="0.1524" layer="16"/>
+<wire x1="48.8442" y1="37.5666" x2="48.8442" y2="18.7452" width="0.1524" layer="16"/>
 <wire x1="57.15" y1="3.5814" x2="57.166" y2="3.556" width="0.1524" layer="16"/>
 <wire x1="48.8442" y1="40.4622" x2="48.895" y2="40.513" width="0.1524" layer="16"/>
@@
 <contactref element="J3" pad="3"/>
 <contactref element="J4" pad="1"/>
+<wire x1="43.5864" y1="37.719" x2="34.417" y2="37.719" width="0.1524" layer="16"/>
+<wire x1="46.3296" y1="40.4622" x2="43.5864" y2="37.719" width="0.1524" layer="16"/>
+<wire x1="46.3296" y1="40.4622" x2="46.355" y2="40.513" width="0.1524" layer="16"/>
 <wire x1="55.0926" y1="8.6106" x2="55.0926" y2="3.5814" width="0.1524" layer="1"/>
 <wire x1="50.2158" y1="13.4874" x2="55.0926" y2="8.6106" width="0.1524" layer="1"/>
@@
 <wire x1="46.355" y1="40.513" x2="50.2158" y2="36.6522" width="0.1524" layer="1"/>
 <wire x1="55.0926" y1="3.5814" x2="55.166" y2="3.556" width="0.1524" layer="1"/>
-<wire x1="43.5864" y1="37.719" x2="34.417" y2="37.719" width="0.1524" layer="16"/>
-<wire x1="46.3296" y1="40.4622" x2="43.5864" y2="37.719" width="0.1524" layer="16"/>
-<wire x1="46.3296" y1="40.4622" x2="46.355" y2="40.513" width="0.1524" layer="16"/>
 </signal>
 <signal name="N$1">
@@
 <wire x1="68.199" y1="22.606" x2="69.977" y2="22.606" width="0.2032" layer="1"/>
 </signal>
-<signal name="N$2" class="1">
+<signal name="V_AC-" class="1">
 <contactref element="R3" pad="2"/>
 <contactref element="J5" pad="+"/>
@@
 <wire x1="60.96" y1="10.8966" x2="60.96" y2="10.922" width="0.8128" layer="1"/>
 <wire x1="56.007" y1="9.6774" x2="55.626" y2="9.525" width="0.8128" layer="1"/>
+<contactref element="R5" pad="2"/>
+<wire x1="52.959" y1="24.003" x2="52.959" y2="24.892" width="0.8128" layer="1"/>
+<wire x1="51.5874" y1="22.6314" x2="52.959" y2="24.003" width="0.8128" layer="1"/>
+<wire x1="51.5874" y1="21.0312" x2="51.5874" y2="22.6314" width="0.8128" layer="1"/>
+<wire x1="52.8066" y1="19.812" x2="51.5874" y2="21.0312" width="0.8128" layer="1"/>
+<wire x1="52.8066" y1="19.812" x2="52.959" y2="19.431" width="0.8128" layer="1"/>
 </signal>
 <signal name="N$3" class="1">
 <contactref element="R2" pad="1"/>
-<contactref element="J5" pad="-2"/>
 <contactref element="B1" pad="AC2"/>
-<wire x1="52.959" y1="21.336" x2="52.959" y2="22.86" width="0.8128" layer="1"/>
+<wire x1="52.959" y1="21.336" x2="52.959" y2="22.098" width="0.8128" layer="1"/>
 <wire x1="55.626" y1="18.669" x2="52.959" y2="21.336" width="0.8128" layer="1"/>
-<wire x1="55.626" y1="14.605" x2="55.626" y2="15.9258" width="0.8128" layer="1"/>
-<wire x1="55.626" y1="15.9258" x2="55.626" y2="18.669" width="0.8128" layer="1"/>
-<wire x1="55.626" y1="15.9258" x2="64.0842" y2="15.9258" width="0.8128" layer="1"/>
-<wire x1="64.0842" y1="15.9258" x2="64.135" y2="15.875" width="0.8128" layer="1"/>
+<wire x1="55.626" y1="14.605" x2="55.626" y2="18.669" width="0.8128" layer="1"/>
+<contactref element="J5" pad="-1"/>
+<wire x1="55.626" y1="14.605" x2="60.833" y2="14.605" width="0.8128" layer="16"/>
+<wire x1="60.833" y1="14.605" x2="61.468" y2="13.97" width="0.8128" layer="16"/>
+<wire x1="61.468" y1="13.97" x2="64.135" y2="13.97" width="0.8128" layer="16"/>
+<wire x1="64.135" y1="13.97" x2="67.183" y2="10.922" width="0.8128" layer="16"/>
 </signal>
 <signal name="N$4" class="1">
 <contactref element="B1" pad="+"/>
 <contactref element="C1" pad="+"/>
-<contactref element="IC1" pad="1"/>
+<contactref element="IC1-D24V5F5" pad="1"/>
 <wire x1="42.9768" y1="9.525" x2="42.9768" y2="9.0678" width="0.8128" layer="1"/>
 <wire x1="48.006" y1="14.5542" x2="42.9768" y2="9.525" width="0.8128" layer="1"/>
@@
 <wire x1="47.4726" y1="14.5542" x2="48.006" y2="14.605" width="0.8128" layer="1"/>
 </signal>
-<signal name="V_AC">
+<signal name="V_AC+">
 <contactref element="R3" pad="1"/>
 <contactref element="R2" pad="2"/>
 <contactref element="J3" pad="10"/>
-<wire x1="60.579" y1="22.86" x2="60.579" y2="19.431" width="0.1524" layer="1"/>
+<wire x1="60.579" y1="22.098" x2="60.579" y2="19.431" width="0.1524" layer="1"/>
 <wire x1="64.0842" y1="40.0812" x2="64.0842" y2="40.4622" width="0.1524" layer="16"/>
-<wire x1="60.579" y1="36.576" x2="64.0842" y2="40.0812" width="0.1524" layer="16"/>
-<wire x1="60.579" y1="22.86" x2="60.579" y2="36.576" width="0.1524" layer="16"/>
+<wire x1="61.5696" y1="37.5666" x2="64.0842" y2="40.0812" width="0.1524" layer="16"/>
+<wire x1="61.5696" y1="23.0886" x2="61.5696" y2="37.5666" width="0.1524" layer="16"/>
+<wire x1="60.579" y1="22.098" x2="61.5696" y2="23.0886" width="0.1524" layer="16"/>
 <wire x1="64.0842" y1="40.4622" x2="64.135" y2="40.513" width="0.1524" layer="16"/>
 </signal>
@@
 <contactref element="J3" pad="6"/>
 </signal>
+<signal name="A2" class="1">
+<contactref element="R5" pad="1"/>
+<contactref element="J3" pad="9"/>
+<wire x1="60.579" y1="39.4716" x2="60.579" y2="24.892" width="0.8128" layer="16"/>
+<wire x1="61.5696" y1="40.4622" x2="60.579" y2="39.4716" width="0.8128" layer="16"/>
+<wire x1="61.5696" y1="40.4622" x2="61.595" y2="40.513" width="0.8128" layer="16"/>
+</signal>
 </signals>

Commit message: Switching to SMD
Parts:
- removed B1: (no value), rectifier:B-DIL
- removed J4: 4P-2.0, Seeed-OPL-Connector:HW4-2.0
- removed X1: STEREOJACK, adafruit:STX3100
- added B2: MB8S, rectifier:SOIC-4
- added J6: ST-PJ-312, Seeed-OPL-Connector:AUDIO6P-SMD-3.5-14.0X6.4X5.0MM
- added J7: H4P-SMD-2.0, Seeed-OPL-Connector:HW4-SMD-2.0
- C1: device adafruit:TT2D4 -> adafruit:153CLV-0405
- C2: device adafruit:TT2D4 -> adafruit:175TMP-0808
- R2, R3, R4, R5: device resistor:0204/7 -> resistor:R0603
- moved R4 1.49 mm to (54.6, 31.8)
- moved C1 1.17 mm to (43.7, 6.86), turned to 0 degrees
- moved R5 1.08 mm to (56.0, 24.1)
- moved R3 0.92 mm to (56.0, 19.9)
- moved C2 0.90 mm to (43.8, 13.8), turned to 180 degrees
- moved R2 0.77 mm to (56.0, 22.0)
Connections:
- net 3V3: now also J7.3; no longer J4.3
- net D1: now also J7.1; no longer J4.1
- net D2: now also J7.2; no longer J4.2
- net GND: now also B2.+, J7.4; no longer B1.-, J4.4
- net I_AC+: now also J6.R; no longer X1.5
- net I_AC-: now also J6.COM2; no longer X1.1
- net N$3: now also B2.~1; no longer B1.AC2
- net N$4: now also B2.-; no longer B1.+
- net V_AC-: now also B2.~2; no longer B1.AC1
Routing:
- net D2: track 58.4 -> 2.54 mm
- net D1: track 56.3 -> 15.6 mm
- net I_AC-: track 30.9 -> 0.00 mm
- net V_AC-: track 23.5 -> 0.03 mm
- net N$3: track 21.7 -> 0.00 mm
- net V_AC+: track 22.6 -> 2.03 mm
- net A2: track 16.0 -> 0.00 mm
- net VIN: track 51.2 -> 35.4 mm
- net N$4: track 15.7 -> 0.53 mm
- net I_AC+: track 12.2 -> 0.00 mm

Commit message: Addded SMD jack and routing, polarity wrong
Parts:
- removed J5: DC-005, Seeed-OPL-Connector:DCJ3P-14.2X11.0X9.0MM
- added J4: (no value), dp_devices:DC_BARREL_JACK_SMD_2MM
- moved B2 16.5 mm to (62.5, 25.9), turned to 0 degrees
- moved PWR 15.5 mm to (54.7, 19.2), turned to 180 degrees
- moved R1 11.1 mm to (57.8, 25.7)
- moved R2 10.6 mm to (66.0, 25.7), turned to 90 degrees
- moved R3 5.72 mm to (55.8, 25.7), turned to 270 degrees
- moved J6 4.83 mm to (70.1, 33.7)
- moved R5 2.96 mm to (53.5, 25.7), turned to 270 degrees
Connections:
- net N$3: now also J4.P2; no longer J5.-1
- net V_AC-: now also J4.P1@2; no longer J5.+
Routing:
- net D2: track 2.54 -> 56.8 mm
- net D1: track 15.6 -> 59.1 mm
- net V_AC-: track 0.03 -> 38.8 mm
- net N$4: track 0.53 -> 38.9 mm, vias 0 -> 1
- net I_AC-: track 0.00 -> 32.2 mm, vias 0 -> 2
- net V_AC+: track 2.03 -> 30.4 mm
- net VIN: track 35.4 -> 59.6 mm
- net A2: track 0.00 -> 17.5 mm, vias 0 -> 1
- net I_AC+: track 0.00 -> 16.6 mm
- net N$3: track 0.00 -> 9.73 mm
- net N$1: track 1.78 -> 8.17 mm
- net 3V3: track 120.6 -> 122.4 mm, vias 0 -> 2
Other:
- board size 73 x 44.7 mm -> 67.6 x 44.7 mm

Commit message: Routed fixed rectifier polarity
Connections:
- net GND: now also B2.-; no longer B2.+
- net N$4: now also B2.+; no longer B2.-
Routing:
- net 3V3: track 122.4 -> 0.00 mm, vias 2 -> 0
- net VIN: track 59.6 -> 0.00 mm
- net D1: track 59.1 -> 0.00 mm
- net D2: track 56.8 -> 0.00 mm
- net N$4: track 38.9 -> 0.00 mm, vias 1 -> 0
- net V_AC-: track 38.8 -> 0.00 mm
- net I_AC-: track 32.2 -> 0.00 mm, vias 2 -> 0
- net V_AC+: track 30.4 -> 0.00 mm
- net A2: track 17.5 -> 0.00 mm, vias 1 -> 0
- net I_AC+: track 16.6 -> 0.00 mm
- net N$3: track 9.73 -> 0.00 mm
- net N$1: track 8.17 -> 0.00 mm
- net D9: track 2.54 -> 0.00 mm
- net D8: track 2.54 -> 0.00 mm
- net D7: track 2.54 -> 0.00 mm
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
Commit message: Routed
Parts:
- moved PWR 5.29 mm to (52.1, 14.6), turned to 270 degrees
- moved R4 1.91 mm to (54.5, 33.7)
- moved J6 0.76 mm to (70.9, 33.7)
- moved C2 0.25 mm to (43.6, 13.8), turned to 0 degrees
Connections:
- net GND: now also J7.SS1, J7.SS2
Routing:
- net 3V3: track 0.00 -> 134.4 mm, vias 0 -> 1
- net D2: track 0.00 -> 57.6 mm
- net VIN: track 0.00 -> 57.3 mm
- net D1: track 0.00 -> 55.0 mm
- net N$4: track 0.00 -> 40.0 mm, vias 0 -> 1
- net I_AC-: track 0.00 -> 29.4 mm, vias 0 -> 1
- net V_AC-: track 0.00 -> 28.1 mm, vias 0 -> 2
- net V_AC+: track 0.00 -> 24.9 mm
- net A2: track 0.00 -> 17.4 mm, vias 0 -> 1
- net I_AC+: track 0.00 -> 16.4 mm
- net N$1: track 0.00 -> 13.4 mm
- net N$3: track 0.00 -> 9.16 mm
- net CMD: track 0.00 -> 2.62 mm
- net A0: track 0.00 -> 2.62 mm
- net RST: track 0.00 -> 2.62 mm
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