File: NodeMCU_Emon.brd (EAGLE design)
At the start: 73 x 44.7 mm, 20 parts, among them IC1-D24V5F5 7805T, J3 10p-2.54, J4 4P-2.0, J5 DC-005, X1 STEREOJACK

Commit message: Changed values
Parts:
- C1: value 10uF -> 100uF
- C2: value 100uF -> 10uF
- R4: value 330R -> 100R
Changed lines of the file:
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@@
 </element>
 <element name="R3" library="resistor" package="0204/7" value="10K" x="56.769" y="19.431" rot="R180"/>
-<element name="R4" library="resistor" package="0204/7" value="330R" x="56.007" y="32.258" rot="R90"/>
+<element name="R4" library="resistor" package="0204/7" value="100R" x="56.007" y="32.258" rot="R90"/>
 <element name="X1" library="adafruit" package="STX3100" value="STEREOJACK" x="71.247" y="32.258" smashed="yes" rot="R180">
 <attribute name="NAME" x="67.103" y="25.373" size="1.27" layer="25" ratio="10" rot="R180"/>
 <attribute name="VALUE" x="69.897" y="39.978" size="1.27" layer="27" ratio="10" rot="R180"/>
 </element>
-<element name="C1" library="adafruit" package="TT2D4" value="10uF" x="42.926" y="7.747" rot="R270"/>
-<element name="C2" library="adafruit" package="TT2D4" value="100uF" x="42.926" y="13.97" rot="R90"/>
+<element name="C1" library="adafruit" package="TT2D4" value="100uF" x="42.926" y="7.747" rot="R270"/>
+<element name="C2" library="adafruit" package="TT2D4" value="10uF" x="42.926" y="13.97" rot="R90"/>
 <element name="IC1-D24V5F5" library="adafruit" package="TO220H" value="7805T" x="45.085" y="30.099" smashed="yes">
 <attribute name="NAME" x="52.197" y="21.209" size="1.778" layer="25" ratio="10" rot="R90"/>
