File: NodeMCU_Emon.sch (EAGLE design)
At the start: 18 parts, among them IC1-D24V5F5 7805T, J3 10p-2.54, J4 4P-2.0, J5 DC-005, X1 STEREOJACK

Commit message: Changed values
Parts:
- C1: value 10uF -> 100uF
- C2: value 100uF -> 10uF
- R4: value 330R -> 100R
Changed lines of the file:
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@@
 <part name="R2" library="resistor" deviceset="R-EU_" device="0204/7" value="100K"/>
 <part name="R3" library="resistor" deviceset="R-EU_" device="0204/7" value="10K"/>
-<part name="R4" library="resistor" deviceset="R-EU_" device="0204/7" value="330R"/>
+<part name="R4" library="resistor" deviceset="R-EU_" device="0204/7" value="100R"/>
 <part name="X1" library="adafruit" deviceset="STEREOJACK" device=""/>
-<part name="C1" library="adafruit" deviceset="CPOL-US" device="TT2D4" value="10uF"/>
-<part name="C2" library="adafruit" deviceset="CPOL-US" device="TT2D4" value="100uF"/>
+<part name="C1" library="adafruit" deviceset="CPOL-US" device="TT2D4" value="100uF"/>
+<part name="C2" library="adafruit" deviceset="CPOL-US" device="TT2D4" value="10uF"/>
 <part name="IC1-D24V5F5" library="adafruit" deviceset="78*" device="T" technology="05"/>
 <part name="B1" library="rectifier" deviceset="B-DIL" device=""/>
