File: NodeMCU_Emon.sch (EAGLE design)
At the start: 17 parts, among them IC1 7805T, J3 10p-2.54, J4 4P-2.0, J5 DC-005, X1 STEREOJACK

Commit message: Added extra resistor to protect ADC
Parts:
- added R5: 10K, resistor:R-EU_0204/7
- C2: value 10uF -> 100uF
- R2: value 22K -> 100K
- renumbered IC1 to IC1-D24V5F5
Connections:
- net V_AC renamed V_AC+
- removed net N$2: B1.AC1, J5.+, R3.2
- new net A2: J3.9, R5.1
- new net V_AC-: B1.AC1, J5.+, R3.2, R5.2
- net GND: no longer J3.9
- net N$3: now also J5.-; no longer J5.CDN
Changed lines of the file:
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@@
 <?xml version="1.0" encoding="utf-8"?>
 <!DOCTYPE eagle SYSTEM "eagle.dtd">
-<eagle version="7.3.0">
+<eagle version="7.1.0">
 <drawing>
 <settings>
@@
 <part name="J3" library="Seeed-OPL-Connector" deviceset="DIP-BLACK-FEMALE-HEADER-VERT(10P-2.54)" device="" value="10p-2.54"/>
 <part name="J5" library="Seeed-OPL-Connector" deviceset="CONN-POWER-JACK-2.1MM(DC-005)" device="" value="DC-005"/>
-<part name="R2" library="resistor" deviceset="R-EU_" device="0204/7" value="22K"/>
+<part name="R2" library="resistor" deviceset="R-EU_" device="0204/7" value="100K"/>
 <part name="R3" library="resistor" deviceset="R-EU_" device="0204/7" value="10K"/>
 <part name="R4" library="resistor" deviceset="R-EU_" device="0204/7" value="330R"/>
 <part name="X1" library="adafruit" deviceset="STEREOJACK" device=""/>
 <part name="C1" library="adafruit" deviceset="CPOL-US" device="TT2D4" value="10uF"/>
-<part name="C2" library="adafruit" deviceset="CPOL-US" device="TT2D4" value="10uF"/>
-<part name="IC1" library="adafruit" deviceset="78*" device="T" technology="05"/>
+<part name="C2" library="adafruit" deviceset="CPOL-US" device="TT2D4" value="100uF"/>
+<part name="IC1-D24V5F5" library="adafruit" deviceset="78*" device="T" technology="05"/>
 <part name="B1" library="rectifier" deviceset="B-DIL" device=""/>
 <part name="U$1" library="Power or GND " deviceset="GND_POWER" device=""/>
 <part name="J4" library="Seeed-OPL-Connector" deviceset="GROVE-CONNECTOR-DIP(4P-2.0)" device="" value="4P-2.0"/>
+<part name="R5" library="resistor" deviceset="R-EU_" device="0204/7" value="10K"/>
 </parts>
 <sheets>
@@
 <instance part="C1" gate="G$1" x="157.48" y="104.14"/>
 <instance part="C2" gate="G$1" x="124.46" y="104.14"/>
-<instance part="IC1" gate="A1" x="142.24" y="109.22" rot="MR0"/>
+<instance part="IC1-D24V5F5" gate="A1" x="142.24" y="109.22" rot="MR0"/>
 <instance part="B1" gate="1" x="177.8" y="104.14" rot="R180"/>
 <instance part="U$1" gate="G$1" x="146.05" y="93.98"/>
 <instance part="J4" gate="G$1" x="157.48" y="160.02" rot="R90"/>
+<instance part="R5" gate="G$1" x="135.89" y="147.828" rot="R270"/>
 </instances>
 <busses>
@@
 <wire x1="124.46" y1="99.06" x2="124.46" y2="93.98" width="0.1524" layer="91"/>
 <wire x1="124.46" y1="93.98" x2="142.24" y2="93.98" width="0.1524" layer="91"/>
-<pinref part="IC1" gate="A1" pin="GND"/>
+<pinref part="IC1-D24V5F5" gate="A1" pin="GND"/>
 <wire x1="142.24" y1="93.98" x2="142.24" y2="101.6" width="0.1524" layer="91"/>
 <pinref part="B1" gate="1" pin="-"/>
@@
 </segment>
 <segment>
-<label x="135.89" y="148.59" size="1.778" layer="95" rot="R270" xref="yes"/>
-<pinref part="J3" gate="G$1" pin="9"/>
-<wire x1="135.89" y1="153.67" x2="135.89" y2="147.32" width="0.1524" layer="91"/>
-</segment>
-<segment>
 <pinref part="J4" gate="G$1" pin="4"/>
 <wire x1="161.29" y1="156.21" x2="161.29" y2="149.86" width="0.1524" layer="91"/>
@@
 </segment>
 <segment>
-<pinref part="IC1" gate="A1" pin="VO"/>
+<pinref part="IC1-D24V5F5" gate="A1" pin="VO"/>
 <pinref part="C2" gate="G$1" pin="+"/>
 <wire x1="132.08" y1="109.22" x2="124.46" y2="109.22" width="0.1524" layer="91"/>
@@
 </segment>
 </net>
-<net name="N$2" class="1">
+<net name="V_AC-" class="1">
 <segment>
 <wire x1="205.74" y1="101.6" x2="205.74" y2="91.44" width="0.1524" layer="91"/>
@@
 <pinref part="B1" gate="1" pin="AC1"/>
 <wire x1="177.8" y1="91.44" x2="177.8" y2="99.06" width="0.1524" layer="91"/>
+<label x="187.96" y="88.9" size="1.778" layer="95"/>
+</segment>
+<segment>
+<label x="135.89" y="138.43" size="1.778" layer="95" rot="R270" xref="yes"/>
+<pinref part="R5" gate="G$1" pin="2"/>
+<wire x1="135.89" y1="142.748" x2="135.89" y2="138.684" width="0.1524" layer="91"/>
 </segment>
 </net>
@@
 <wire x1="177.8" y1="116.84" x2="195.58" y2="116.84" width="0.1524" layer="91"/>
 <wire x1="195.58" y1="116.84" x2="208.28" y2="116.84" width="0.1524" layer="91"/>
-<wire x1="208.28" y1="116.84" x2="208.28" y2="104.14" width="0.1524" layer="91"/>
+<wire x1="208.28" y1="116.84" x2="208.28" y2="106.68" width="0.1524" layer="91"/>
 <junction x="195.58" y="116.84"/>
-<pinref part="J5" gate="JACK" pin="CDN"/>
-<wire x1="209.55" y1="104.14" x2="208.28" y2="104.14" width="0.1524" layer="91"/>
 <pinref part="B1" gate="1" pin="AC2"/>
 <wire x1="177.8" y1="116.84" x2="177.8" y2="109.22" width="0.1524" layer="91"/>
+<pinref part="J5" gate="JACK" pin="-"/>
+<wire x1="209.55" y1="106.68" x2="208.28" y2="106.68" width="0.1524" layer="91"/>
 </segment>
 </net>
@@
 <wire x1="157.48" y1="109.22" x2="152.4" y2="109.22" width="0.1524" layer="91"/>
 <junction x="157.48" y="109.22"/>
-<pinref part="IC1" gate="A1" pin="VI"/>
-</segment>
-</net>
-<net name="V_AC" class="0">
+<pinref part="IC1-D24V5F5" gate="A1" pin="VI"/>
+</segment>
+</net>
+<net name="V_AC+" class="0">
 <segment>
 <pinref part="R3" gate="G$1" pin="1"/>
@@
 </segment>
 </net>
+<net name="A2" class="1">
+<segment>
+<pinref part="J3" gate="G$1" pin="9"/>
+<wire x1="135.89" y1="153.67" x2="135.89" y2="152.908" width="0.1524" layer="91"/>
+<pinref part="R5" gate="G$1" pin="1"/>
+</segment>
+</net>

Commit message: Switching to SMD
Parts:
- removed B1: (no value), rectifier:B-DIL
- removed J4: 4P-2.0, Seeed-OPL-Connector:GROVE-CONNECTOR-DIP(4P-2.0)
- removed X1: STEREOJACK, adafruit:STEREOJACK
- added B2: MB8S, rectifier:MB8S
- added J6: ST-PJ-312, Seeed-OPL-Connector:AUDIO-JACK-6P-SMD(ST-PJ-312)
- added J7: H4P-SMD-2.0, Seeed-OPL-Connector:GROVE-CONNECTOR-SMD(4+2P-2.0)
- C1: device adafruit:CPOL-USTT2D4 -> adafruit:CPOL-US153CLV-0405
- C2: device adafruit:CPOL-USTT2D4 -> adafruit:CPOL-US175TMP-0808
- R2, R3, R4, R5: device resistor:R-EU_0204/7 -> resistor:R-EU_R0603
Connections:
- net 3V3: now also J7.3; no longer J4.3
- net D1: now also J7.1; no longer J4.1
- net D2: now also J7.2; no longer J4.2
- net GND: now also B2.+, J7.4; no longer B1.-, J4.4
- net I_AC+: now also J6.R; no longer X1.5
- net I_AC-: now also J6.COM2; no longer X1.1
- net N$3: now also B2.AC1; no longer B1.AC2
- net N$4: now also B2.-; no longer B1.+
- net V_AC-: now also B2.AC2; no longer B1.AC1

Commit message: Addded SMD jack and routing, polarity wrong
Parts:
- removed J5: DC-005, Seeed-OPL-Connector:CONN-POWER-JACK-2.1MM(DC-005)
- added J4: (no value), dp_devices:CON_DC_M-DC_SMD
Connections:
- net N$3: now also J4.P2; no longer J5.-
- net V_AC-: now also J4.P1; no longer J5.+
Changed lines of the file:
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@@
 <grid distance="0.1" unitdist="inch" unit="inch" style="lines" multiple="1" display="no" altdistance="0.01" altunitdist="inch" altunit="inch"/>
 <layers>
-<layer number="1" name="Top" color="4" fill="1" visible="yes" active="no"/>
-<layer number="2" name="Route2" color="1" fill="3" visible="yes" active="no"/>
-<layer number="3" name="Route3" color="4" fill="3" visible="yes" active="no"/>
-<layer number="4" name="Route4" color="1" fill="4" visible="yes" active="no"/>
-<layer number="5" name="Route5" color="4" fill="4" visible="yes" active="no"/>
-<layer number="6" name="Route6" color="1" fill="8" visible="yes" active="no"/>
-<layer number="7" name="Route7" color="4" fill="8" visible="yes" active="no"/>
-<layer number="8" name="Route8" color="1" fill="2" visible="yes" active="no"/>
-<layer number="9" name="Route9" color="4" fill="2" visible="yes" active="no"/>
-<layer number="10" name="Route10" color="1" fill="7" visible="yes" active="no"/>
-<layer number="11" name="Route11" color="4" fill="7" visible="yes" active="no"/>
-<layer number="12" name="Route12" color="1" fill="5" visible="yes" active="no"/>
-<layer number="13" name="Route13" color="4" fill="5" visible="yes" active="no"/>
-<layer number="14" name="Route14" color="1" fill="6" visible="yes" active="no"/>
-<layer number="15" name="Route15" color="4" fill="6" visible="yes" active="no"/>
-<layer number="16" name="Bottom" color="1" fill="1" visible="yes" active="no"/>
-<layer number="17" name="Pads" color="2" fill="1" visible="yes" active="no"/>
-<layer number="18" name="Vias" color="2" fill="1" visible="yes" active="no"/>
-<layer number="19" name="Unrouted" color="6" fill="1" visible="yes" active="no"/>
-<layer number="20" name="Dimension" color="5" fill="1" visible="yes" active="no"/>
-<layer number="21" name="tPlace" color="7" fill="1" visible="yes" active="no"/>
-<layer number="22" name="bPlace" color="3" fill="1" visible="yes" active="no"/>
-<layer number="23" name="tOrigins" color="15" fill="1" visible="yes" active="no"/>
-<layer number="24" name="bOrigins" color="3" fill="1" visible="yes" active="no"/>
-<layer number="25" name="tNames" color="7" fill="1" visible="yes" active="no"/>
-<layer number="26" name="bNames" color="3" fill="1" visible="yes" active="no"/>
-<layer number="27" name="tValues" color="7" fill="1" visible="yes" active="no"/>
-<layer number="28" name="bValues" color="7" fill="1" visible="yes" active="no"/>
+<layer number="1" name="Top" color="4" fill="1" visible="no" active="no"/>
+<layer number="2" name="Route2" color="1" fill="3" visible="no" active="no"/>
+<layer number="3" name="Route3" color="4" fill="3" visible="no" active="no"/>
+<layer number="4" name="Route4" color="1" fill="4" visible="no" active="no"/>
+<layer number="5" name="Route5" color="4" fill="4" visible="no" active="no"/>
+<layer number="6" name="Route6" color="1" fill="8" visible="no" active="no"/>
+<layer number="7" name="Route7" color="4" fill="8" visible="no" active="no"/>
+<layer number="8" name="Route8" color="1" fill="2" visible="no" active="no"/>
+<layer number="9" name="Route9" color="4" fill="2" visible="no" active="no"/>
+<layer number="10" name="Route10" color="1" fill="7" visible="no" active="no"/>
+<layer number="11" name="Route11" color="4" fill="7" visible="no" active="no"/>
+<layer number="12" name="Route12" color="1" fill="5" visible="no" active="no"/>
+<layer number="13" name="Route13" color="4" fill="5" visible="no" active="no"/>
+<layer number="14" name="Route14" color="1" fill="6" visible="no" active="no"/>
+<layer number="15" name="Route15" color="4" fill="6" visible="no" active="no"/>
+<layer number="16" name="Bottom" color="1" fill="1" visible="no" active="no"/>
+<layer number="17" name="Pads" color="2" fill="1" visible="no" active="no"/>
+<layer number="18" name="Vias" color="2" fill="1" visible="no" active="no"/>
+<layer number="19" name="Unrouted" color="6" fill="1" visible="no" active="no"/>
+<layer number="20" name="Dimension" color="5" fill="1" visible="no" active="no"/>
+<layer number="21" name="tPlace" color="7" fill="1" visible="no" active="no"/>
+<layer number="22" name="bPlace" color="3" fill="1" visible="no" active="no"/>
+<layer number="23" name="tOrigins" color="15" fill="1" visible="no" active="no"/>
+<layer number="24" name="bOrigins" color="3" fill="1" visible="no" active="no"/>
+<layer number="25" name="tNames" color="7" fill="1" visible="no" active="no"/>
+<layer number="26" name="bNames" color="3" fill="1" visible="no" active="no"/>
+<layer number="27" name="tValues" color="7" fill="1" visible="no" active="no"/>
+<layer number="28" name="bValues" color="7" fill="1" visible="no" active="no"/>
 <layer number="29" name="tStop" color="7" fill="3" visible="no" active="no"/>
 <layer number="30" name="bStop" color="3" fill="6" visible="no" active="no"/>
@@
 <layer number="35" name="tGlue" color="7" fill="4" visible="no" active="no"/>
 <layer number="36" name="bGlue" color="3" fill="5" visible="no" active="no"/>
-<layer number="37" name="tTest" color="7" fill="1" visible="yes" active="no"/>
-<layer number="38" name="bTest" color="3" fill="1" visible="yes" active="no"/>
+<layer number="37" name="tTest" color="7" fill="1" visible="no" active="no"/>
+<layer number="38" name="bTest" color="3" fill="1" visible="no" active="no"/>
 <layer number="39" name="tKeepout" color="4" fill="11" visible="no" active="no"/>
 <layer number="40" name="bKeepout" color="1" fill="11" visible="no" active="no"/>
@@
 <layer number="44" name="Drills" color="7" fill="1" visible="no" active="no"/>
 <layer number="45" name="Holes" color="7" fill="1" visible="no" active="no"/>
-<layer number="46" name="Milling" color="3" fill="1" visible="yes" active="no"/>
-<layer number="47" name="Measures" color="7" fill="1" visible="yes" active="no"/>
-<layer number="48" name="Document" color="7" fill="1" visible="yes" active="no"/>
-<layer number="49" name="Reference" color="7" fill="1" visible="yes" active="no"/>
-<layer number="50" name="dxf" color="7" fill="1" visible="yes" active="no"/>
-<layer number="51" name="tDocu" color="7" fill="1" visible="yes" active="no"/>
-<layer number="52" name="bDocu" color="7" fill="1" visible="yes" active="no"/>
-<layer number="53" name="tGND_GNDA" color="7" fill="9" visible="yes" active="no"/>
-<layer number="54" name="bGND_GNDA" color="1" fill="9" visible="yes" active="no"/>
-<layer number="56" name="wert" color="7" fill="1" visible="yes" active="no"/>
-<layer number="57" name="tCAD" color="7" fill="1" visible="yes" active="no"/>
+<layer number="46" name="Milling" color="3" fill="1" visible="no" active="no"/>
+<layer number="47" name="Measures" color="7" fill="1" visible="no" active="no"/>
+<layer number="48" name="Document" color="7" fill="1" visible="no" active="no"/>
+<layer number="49" name="Reference" color="7" fill="1" visible="no" active="no"/>
+<layer number="50" name="dxf" color="7" fill="1" visible="no" active="no"/>
+<layer number="51" name="tDocu" color="7" fill="1" visible="no" active="no"/>
+<layer number="52" name="bDocu" color="7" fill="1" visible="no" active="no"/>
+<layer number="53" name="tGND_GNDA" color="7" fill="9" visible="no" active="no"/>
+<layer number="54" name="bGND_GNDA" color="1" fill="9" visible="no" active="no"/>
+<layer number="56" name="wert" color="7" fill="1" visible="no" active="no"/>
+<layer number="57" name="tCAD" color="7" fill="1" visible="no" active="no"/>
 <layer number="90" name="Modules" color="5" fill="1" visible="yes" active="yes"/>
 <layer number="91" name="Nets" color="2" fill="1" visible="yes" active="yes"/>
@@
 <part name="U$4" library="Power or GND " deviceset="GND_POWER" device=""/>
 <part name="J3" library="Seeed-OPL-Connector" deviceset="DIP-BLACK-FEMALE-HEADER-VERT(10P-2.54)" device="" value="10p-2.54"/>
-<part name="J5" library="Seeed-OPL-Connector" deviceset="CONN-POWER-JACK-2.1MM(DC-005)" device="" value="DC-005"/>
 <part name="R2" library="resistor" deviceset="R-EU_" device="R0603" value="100K"/>
 <part name="R3" library="resistor" deviceset="R-EU_" device="R0603" value="10K"/>
@@
 <part name="J7" library="Seeed-OPL-Connector" deviceset="GROVE-CONNECTOR-SMD(4+2P-2.0)" device="" value="H4P-SMD-2.0"/>
 <part name="B2" library="rectifier" deviceset="MB*S" device="" technology="8"/>
+<part name="J4" library="dp_devices" deviceset="CON_DC_M" device="-DC_SMD"/>
 </parts>
 <sheets>
@@
 <instance part="U$4" gate="G$1" x="74.93" y="30.48"/>
 <instance part="J3" gate="G$1" x="127" y="160.02" rot="R90"/>
-<instance part="J5" gate="JACK" x="215.9" y="104.14" rot="R180"/>
 <instance part="R2" gate="G$1" x="195.58" y="111.76" rot="R270"/>
 <instance part="R3" gate="G$1" x="195.58" y="96.52" rot="R270"/>
@@
 <instance part="J7" gate="G$1" x="157.48" y="162.56" rot="R90"/>
 <instance part="B2" gate="G$1" x="177.8" y="104.14"/>
+<instance part="J4" gate="J" x="213.36" y="104.14" rot="R180"/>
 </instances>
 <busses>
@@
 <wire x1="195.58" y1="91.44" x2="177.8" y2="91.44" width="0.1524" layer="91"/>
 <junction x="195.58" y="91.44"/>
-<wire x1="205.74" y1="101.6" x2="209.55" y2="101.6" width="0.1524" layer="91"/>
-<pinref part="J5" gate="JACK" pin="+"/>
+<wire x1="205.74" y1="101.6" x2="208.28" y2="101.6" width="0.1524" layer="91"/>
 <wire x1="177.8" y1="91.44" x2="177.8" y2="99.06" width="0.1524" layer="91"/>
 <label x="187.96" y="88.9" size="1.778" layer="95"/>
 <pinref part="B2" gate="G$1" pin="AC2"/>
+<pinref part="J4" gate="J" pin="P1"/>
 </segment>
 <segment>
@@
 <junction x="195.58" y="116.84"/>
 <wire x1="177.8" y1="116.84" x2="177.8" y2="109.22" width="0.1524" layer="91"/>
-<pinref part="J5" gate="JACK" pin="-"/>
-<wire x1="209.55" y1="106.68" x2="208.28" y2="106.68" width="0.1524" layer="91"/>
 <pinref part="B2" gate="G$1" pin="AC1"/>
-</segment>
-</net>
+<pinref part="J4" gate="J" pin="P2"/>
+</segment>
+</net>

Commit message: Routed fixed rectifier polarity
Connections:
- net GND: now also B2.-; no longer B2.+
- net N$4: now also B2.+; no longer B2.-
Changed lines of the file:
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@@
 <instance part="J6" gate="G$1" x="223.52" y="132.08"/>
 <instance part="J7" gate="G$1" x="157.48" y="162.56" rot="R90"/>
-<instance part="B2" gate="G$1" x="177.8" y="104.14"/>
+<instance part="B2" gate="G$1" x="177.8" y="104.14" rot="MR0"/>
 <instance part="J4" gate="J" x="213.36" y="104.14" rot="R180"/>
 </instances>
@@
 <pinref part="IC1-D24V5F5" gate="A1" pin="GND"/>
 <wire x1="142.24" y1="93.98" x2="142.24" y2="101.6" width="0.1524" layer="91"/>
-<wire x1="182.88" y1="104.14" x2="185.42" y2="104.14" width="0.1524" layer="91"/>
 <wire x1="185.42" y1="104.14" x2="185.42" y2="93.98" width="0.1524" layer="91"/>
 <wire x1="185.42" y1="93.98" x2="157.48" y2="93.98" width="0.1524" layer="91"/>
@@
 <pinref part="U$1" gate="G$1" pin="GND"/>
 <junction x="146.05" y="93.98"/>
-<pinref part="B2" gate="G$1" pin="+"/>
+<pinref part="B2" gate="G$1" pin="-"/>
+<wire x1="182.88" y1="104.14" x2="185.42" y2="104.14" width="0.1524" layer="91"/>
 </segment>
 <segment>
@@
 <net name="N$4" class="1">
 <segment>
-<wire x1="172.72" y1="104.14" x2="165.1" y2="104.14" width="0.1524" layer="91"/>
 <wire x1="165.1" y1="104.14" x2="165.1" y2="109.22" width="0.1524" layer="91"/>
 <pinref part="C1" gate="G$1" pin="+"/>
@@
 <junction x="157.48" y="109.22"/>
 <pinref part="IC1-D24V5F5" gate="A1" pin="VI"/>
-<pinref part="B2" gate="G$1" pin="-"/>
-</segment>
-</net>
+<pinref part="B2" gate="G$1" pin="+"/>
+<wire x1="165.1" y1="104.14" x2="172.72" y2="104.14" width="0.1524" layer="91"/>
+</segment>
+</net>

Commit message: Routed
Connections:
- net GND: now also J7.SS1, J7.SS2
Changed lines of the file:
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@@
 <label x="161.29" y="152.4" size="1.778" layer="95" rot="R270" xref="yes"/>
 <pinref part="J7" gate="G$1" pin="4"/>
-<wire x1="161.29" y1="157.48" x2="161.29" y2="149.86" width="0.1524" layer="91"/>
+<wire x1="161.29" y1="157.48" x2="161.29" y2="154.94" width="0.1524" layer="91"/>
+<pinref part="J7" gate="G$1" pin="SS1"/>
+<wire x1="161.29" y1="154.94" x2="161.29" y2="149.86" width="0.1524" layer="91"/>
+<wire x1="149.86" y1="162.56" x2="144.78" y2="162.56" width="0.1524" layer="91"/>
+<wire x1="144.78" y1="162.56" x2="144.78" y2="154.94" width="0.1524" layer="91"/>
+<wire x1="144.78" y1="154.94" x2="161.29" y2="154.94" width="0.1524" layer="91"/>
+<junction x="161.29" y="154.94"/>
+<pinref part="J7" gate="G$1" pin="SS2"/>
+<wire x1="165.1" y1="162.56" x2="167.64" y2="162.56" width="0.1524" layer="91"/>
+<wire x1="167.64" y1="162.56" x2="167.64" y2="154.94" width="0.1524" layer="91"/>
+<wire x1="167.64" y1="154.94" x2="161.29" y2="154.94" width="0.1524" layer="91"/>
 </segment>
 </net>
