File: NodeMCU_Emon.sch (EAGLE design)
At the start: 18 parts, among them IC1-D24V5F5 7805T, J3 10p-2.54, J6 ST-PJ-312, J7 H4P-SMD-2.0

Commit message: Finished routing and fixups
Parts:
- C1: value 10uF -> 100uF; device adafruit:CPOL-US153CLV-0405 -> adafruit:CPOL-US175TMP-0808
- C2: value 100uF -> 10uF; device adafruit:CPOL-US175TMP-0808 -> adafruit:CPOL-US153CLV-0405
- R4: value 330R -> 100R
Connections:
- net I_AC+: now also J6.COM1; no longer J6.R
- net I_AC-: now also J6.L; no longer J6.COM2
Changed lines of the file:
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@@
 <grid distance="0.1" unitdist="inch" unit="inch" style="lines" multiple="1" display="no" altdistance="0.01" altunitdist="inch" altunit="inch"/>
 <layers>
-<layer number="1" name="Top" color="4" fill="1" visible="no" active="no"/>
-<layer number="2" name="Route2" color="1" fill="3" visible="no" active="no"/>
-<layer number="3" name="Route3" color="4" fill="3" visible="no" active="no"/>
-<layer number="4" name="Route4" color="1" fill="4" visible="no" active="no"/>
-<layer number="5" name="Route5" color="4" fill="4" visible="no" active="no"/>
-<layer number="6" name="Route6" color="1" fill="8" visible="no" active="no"/>
-<layer number="7" name="Route7" color="4" fill="8" visible="no" active="no"/>
-<layer number="8" name="Route8" color="1" fill="2" visible="no" active="no"/>
-<layer number="9" name="Route9" color="4" fill="2" visible="no" active="no"/>
-<layer number="10" name="Route10" color="1" fill="7" visible="no" active="no"/>
-<layer number="11" name="Route11" color="4" fill="7" visible="no" active="no"/>
-<layer number="12" name="Route12" color="1" fill="5" visible="no" active="no"/>
-<layer number="13" name="Route13" color="4" fill="5" visible="no" active="no"/>
-<layer number="14" name="Route14" color="1" fill="6" visible="no" active="no"/>
-<layer number="15" name="Route15" color="4" fill="6" visible="no" active="no"/>
-<layer number="16" name="Bottom" color="1" fill="1" visible="no" active="no"/>
-<layer number="17" name="Pads" color="2" fill="1" visible="no" active="no"/>
-<layer number="18" name="Vias" color="2" fill="1" visible="no" active="no"/>
-<layer number="19" name="Unrouted" color="6" fill="1" visible="no" active="no"/>
-<layer number="20" name="Dimension" color="5" fill="1" visible="no" active="no"/>
-<layer number="21" name="tPlace" color="7" fill="1" visible="no" active="no"/>
-<layer number="22" name="bPlace" color="3" fill="1" visible="no" active="no"/>
-<layer number="23" name="tOrigins" color="15" fill="1" visible="no" active="no"/>
-<layer number="24" name="bOrigins" color="3" fill="1" visible="no" active="no"/>
-<layer number="25" name="tNames" color="7" fill="1" visible="no" active="no"/>
-<layer number="26" name="bNames" color="3" fill="1" visible="no" active="no"/>
-<layer number="27" name="tValues" color="7" fill="1" visible="no" active="no"/>
-<layer number="28" name="bValues" color="7" fill="1" visible="no" active="no"/>
+<layer number="1" name="Top" color="4" fill="1" visible="yes" active="no"/>
+<layer number="2" name="Route2" color="1" fill="3" visible="yes" active="no"/>
+<layer number="3" name="Route3" color="4" fill="3" visible="yes" active="no"/>
+<layer number="4" name="Route4" color="1" fill="4" visible="yes" active="no"/>
+<layer number="5" name="Route5" color="4" fill="4" visible="yes" active="no"/>
+<layer number="6" name="Route6" color="1" fill="8" visible="yes" active="no"/>
+<layer number="7" name="Route7" color="4" fill="8" visible="yes" active="no"/>
+<layer number="8" name="Route8" color="1" fill="2" visible="yes" active="no"/>
+<layer number="9" name="Route9" color="4" fill="2" visible="yes" active="no"/>
+<layer number="10" name="Route10" color="1" fill="7" visible="yes" active="no"/>
+<layer number="11" name="Route11" color="4" fill="7" visible="yes" active="no"/>
+<layer number="12" name="Route12" color="1" fill="5" visible="yes" active="no"/>
+<layer number="13" name="Route13" color="4" fill="5" visible="yes" active="no"/>
+<layer number="14" name="Route14" color="1" fill="6" visible="yes" active="no"/>
+<layer number="15" name="Route15" color="4" fill="6" visible="yes" active="no"/>
+<layer number="16" name="Bottom" color="1" fill="1" visible="yes" active="no"/>
+<layer number="17" name="Pads" color="2" fill="1" visible="yes" active="no"/>
+<layer number="18" name="Vias" color="2" fill="1" visible="yes" active="no"/>
+<layer number="19" name="Unrouted" color="6" fill="1" visible="yes" active="no"/>
+<layer number="20" name="Dimension" color="5" fill="1" visible="yes" active="no"/>
+<layer number="21" name="tPlace" color="7" fill="1" visible="yes" active="no"/>
+<layer number="22" name="bPlace" color="3" fill="1" visible="yes" active="no"/>
+<layer number="23" name="tOrigins" color="15" fill="1" visible="yes" active="no"/>
+<layer number="24" name="bOrigins" color="3" fill="1" visible="yes" active="no"/>
+<layer number="25" name="tNames" color="7" fill="1" visible="yes" active="no"/>
+<layer number="26" name="bNames" color="3" fill="1" visible="yes" active="no"/>
+<layer number="27" name="tValues" color="7" fill="1" visible="yes" active="no"/>
+<layer number="28" name="bValues" color="7" fill="1" visible="yes" active="no"/>
 <layer number="29" name="tStop" color="7" fill="3" visible="no" active="no"/>
 <layer number="30" name="bStop" color="3" fill="6" visible="no" active="no"/>
@@
 <layer number="35" name="tGlue" color="7" fill="4" visible="no" active="no"/>
 <layer number="36" name="bGlue" color="3" fill="5" visible="no" active="no"/>
-<layer number="37" name="tTest" color="7" fill="1" visible="no" active="no"/>
-<layer number="38" name="bTest" color="3" fill="1" visible="no" active="no"/>
+<layer number="37" name="tTest" color="7" fill="1" visible="yes" active="no"/>
+<layer number="38" name="bTest" color="3" fill="1" visible="yes" active="no"/>
 <layer number="39" name="tKeepout" color="4" fill="11" visible="no" active="no"/>
 <layer number="40" name="bKeepout" color="1" fill="11" visible="no" active="no"/>
@@
 <layer number="44" name="Drills" color="7" fill="1" visible="no" active="no"/>
 <layer number="45" name="Holes" color="7" fill="1" visible="no" active="no"/>
-<layer number="46" name="Milling" color="3" fill="1" visible="no" active="no"/>
-<layer number="47" name="Measures" color="7" fill="1" visible="no" active="no"/>
-<layer number="48" name="Document" color="7" fill="1" visible="no" active="no"/>
-<layer number="49" name="Reference" color="7" fill="1" visible="no" active="no"/>
-<layer number="50" name="dxf" color="7" fill="1" visible="no" active="no"/>
-<layer number="51" name="tDocu" color="7" fill="1" visible="no" active="no"/>
-<layer number="52" name="bDocu" color="7" fill="1" visible="no" active="no"/>
-<layer number="53" name="tGND_GNDA" color="7" fill="9" visible="no" active="no"/>
-<layer number="54" name="bGND_GNDA" color="1" fill="9" visible="no" active="no"/>
-<layer number="56" name="wert" color="7" fill="1" visible="no" active="no"/>
-<layer number="57" name="tCAD" color="7" fill="1" visible="no" active="no"/>
+<layer number="46" name="Milling" color="3" fill="1" visible="yes" active="no"/>
+<layer number="47" name="Measures" color="7" fill="1" visible="yes" active="no"/>
+<layer number="48" name="Document" color="7" fill="1" visible="yes" active="no"/>
+<layer number="49" name="Reference" color="7" fill="1" visible="yes" active="no"/>
+<layer number="50" name="dxf" color="7" fill="1" visible="yes" active="no"/>
+<layer number="51" name="tDocu" color="7" fill="1" visible="yes" active="no"/>
+<layer number="52" name="bDocu" color="7" fill="1" visible="yes" active="no"/>
+<layer number="53" name="tGND_GNDA" color="7" fill="9" visible="yes" active="no"/>
+<layer number="54" name="bGND_GNDA" color="1" fill="9" visible="yes" active="no"/>
+<layer number="56" name="wert" color="7" fill="1" visible="yes" active="no"/>
+<layer number="57" name="tCAD" color="7" fill="1" visible="yes" active="no"/>
 <layer number="90" name="Modules" color="5" fill="1" visible="yes" active="yes"/>
 <layer number="91" name="Nets" color="2" fill="1" visible="yes" active="yes"/>
@@
 <part name="R2" library="resistor" deviceset="R-EU_" device="R0603" value="100K"/>
 <part name="R3" library="resistor" deviceset="R-EU_" device="R0603" value="10K"/>
-<part name="R4" library="resistor" deviceset="R-EU_" device="R0603" value="330R"/>
-<part name="C1" library="adafruit" deviceset="CPOL-US" device="153CLV-0405" value="10uF"/>
-<part name="C2" library="adafruit" deviceset="CPOL-US" device="175TMP-0808" value="100uF"/>
+<part name="R4" library="resistor" deviceset="R-EU_" device="R0603" value="100R"/>
+<part name="C1" library="adafruit" deviceset="CPOL-US" device="175TMP-0808" value="100uF"/>
+<part name="C2" library="adafruit" deviceset="CPOL-US" device="153CLV-0405" value="10uF"/>
 <part name="IC1-D24V5F5" library="adafruit" deviceset="78*" device="T" technology="05"/>
 <part name="U$1" library="Power or GND " deviceset="GND_POWER" device=""/>
@@
 <junction x="196.85" y="123.19"/>
 <label x="186.69" y="123.19" size="1.778" layer="95"/>
-<wire x1="203.2" y1="119.38" x2="234.95" y2="119.38" width="0.1524" layer="91"/>
 <wire x1="203.2" y1="123.19" x2="203.2" y2="119.38" width="0.1524" layer="91"/>
-<wire x1="234.95" y1="121.92" x2="234.95" y2="119.38" width="0.1524" layer="91"/>
-<pinref part="J6" gate="G$1" pin="COM2"/>
+<pinref part="J6" gate="G$1" pin="L"/>
+<wire x1="203.2" y1="119.38" x2="217.17" y2="119.38" width="0.1524" layer="91"/>
+<wire x1="217.17" y1="119.38" x2="217.17" y2="121.92" width="0.1524" layer="91"/>
 </segment>
 <segment>
@@
 <label x="186.69" y="133.35" size="1.778" layer="95"/>
 <wire x1="203.2" y1="133.35" x2="203.2" y2="148.082" width="0.1524" layer="91"/>
-<wire x1="227.33" y1="142.24" x2="227.33" y2="148.082" width="0.1524" layer="91"/>
-<wire x1="227.33" y1="148.082" x2="203.2" y2="148.082" width="0.1524" layer="91"/>
-<pinref part="J6" gate="G$1" pin="R"/>
-</segment>
-<segment>
+<wire x1="232.41" y1="148.082" x2="203.2" y2="148.082" width="0.1524" layer="91"/>
+<pinref part="J6" gate="G$1" pin="COM1"/>
+<wire x1="232.41" y1="142.24" x2="232.41" y2="148.082" width="0.1524" layer="91"/>
+</segment>
+<segment>

Commit message: Changed to XP Power SR05 footprint
Parts:
- removed IC1-D24V5F5: 7805T, adafruit:7805T
- added U1: SR05, Seeed-OPL-ic:PMIC-L7805CV-DG(TO-220)ALT
Connections:
- net GND: now also U1.GND; no longer IC1-D24V5F5.GND
- net N$4: now also U1.IN; no longer IC1-D24V5F5.VI
- net VIN: now also U1.OUT; no longer IC1-D24V5F5.VO
Changed lines of the file:
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@@
 <part name="C1" library="adafruit" deviceset="CPOL-US" device="175TMP-0808" value="100uF"/>
 <part name="C2" library="adafruit" deviceset="CPOL-US" device="153CLV-0405" value="10uF"/>
-<part name="IC1-D24V5F5" library="adafruit" deviceset="78*" device="T" technology="05"/>
 <part name="U$1" library="Power or GND " deviceset="GND_POWER" device=""/>
 <part name="R5" library="resistor" deviceset="R-EU_" device="R0603" value="10K"/>
@@
 <part name="B2" library="rectifier" deviceset="MB*S" device="" technology="8"/>
 <part name="J4" library="dp_devices" deviceset="CON_DC_M" device="-DC_SMD"/>
+<part name="U1" library="Seeed-OPL-ic" deviceset="PMIC-L7805CV-DG(TO-220)" device="ALT" value="SR05"/>
 </parts>
 <sheets>
@@
 <instance part="C1" gate="G$1" x="157.48" y="104.14"/>
 <instance part="C2" gate="G$1" x="124.46" y="104.14"/>
-<instance part="IC1-D24V5F5" gate="A1" x="142.24" y="109.22" rot="MR0"/>
 <instance part="U$1" gate="G$1" x="146.05" y="93.98"/>
 <instance part="R5" gate="G$1" x="135.89" y="147.828" rot="R270"/>
@@
 <instance part="B2" gate="G$1" x="177.8" y="104.14" rot="MR0"/>
 <instance part="J4" gate="J" x="213.36" y="104.14" rot="R180"/>
+<instance part="U1" gate="G$1" x="142.24" y="109.22" rot="MR0"/>
 </instances>
 <busses>
@@
 <wire x1="124.46" y1="99.06" x2="124.46" y2="93.98" width="0.1524" layer="91"/>
 <wire x1="124.46" y1="93.98" x2="142.24" y2="93.98" width="0.1524" layer="91"/>
-<pinref part="IC1-D24V5F5" gate="A1" pin="GND"/>
-<wire x1="142.24" y1="93.98" x2="142.24" y2="101.6" width="0.1524" layer="91"/>
+<wire x1="142.24" y1="93.98" x2="142.24" y2="100.33" width="0.1524" layer="91"/>
 <wire x1="185.42" y1="104.14" x2="185.42" y2="93.98" width="0.1524" layer="91"/>
 <wire x1="185.42" y1="93.98" x2="157.48" y2="93.98" width="0.1524" layer="91"/>
@@
 <pinref part="B2" gate="G$1" pin="-"/>
 <wire x1="182.88" y1="104.14" x2="185.42" y2="104.14" width="0.1524" layer="91"/>
+<pinref part="U1" gate="G$1" pin="GND"/>
 </segment>
 <segment>
@@
 </segment>
 <segment>
-<pinref part="IC1-D24V5F5" gate="A1" pin="VO"/>
 <pinref part="C2" gate="G$1" pin="+"/>
-<wire x1="132.08" y1="109.22" x2="124.46" y2="109.22" width="0.1524" layer="91"/>
+<wire x1="130.81" y1="109.22" x2="124.46" y2="109.22" width="0.1524" layer="91"/>
 <wire x1="124.46" y1="109.22" x2="124.46" y2="106.68" width="0.1524" layer="91"/>
 <wire x1="124.46" y1="109.22" x2="116.84" y2="109.22" width="0.1524" layer="91"/>
 <junction x="124.46" y="109.22"/>
 <label x="116.84" y="109.22" size="1.778" layer="95"/>
+<pinref part="U1" gate="G$1" pin="OUT"/>
 </segment>
 </net>
@@
 <wire x1="165.1" y1="109.22" x2="157.48" y2="109.22" width="0.1524" layer="91"/>
 <wire x1="157.48" y1="109.22" x2="157.48" y2="106.68" width="0.1524" layer="91"/>
-<wire x1="157.48" y1="109.22" x2="152.4" y2="109.22" width="0.1524" layer="91"/>
+<wire x1="157.48" y1="109.22" x2="153.67" y2="109.22" width="0.1524" layer="91"/>
 <junction x="157.48" y="109.22"/>
-<pinref part="IC1-D24V5F5" gate="A1" pin="VI"/>
 <pinref part="B2" gate="G$1" pin="+"/>
 <wire x1="165.1" y1="104.14" x2="172.72" y2="104.14" width="0.1524" layer="91"/>
-</segment>
-</net>
+<pinref part="U1" gate="G$1" pin="IN"/>
+</segment>
+</net>
